File: Circuit/boneIO - relay board 24x10A/boneIO - relay board.kicad_pcb (KiCad board)
At the start: 2 copper layers, 197 x 102 mm, 76 parts, among them J1 Screw_Terminal_01x04, J10 Screw_Terminal_01x04, J11 Screw_Terminal_01x04, J12 Screw_Terminal_01x04, J13 Screw_Terminal_01x04, J2 Screw_Terminal_01x04, J3 Conn_02x04_Odd_Even, J4 Screw_Terminal_01x04, J5 Screw_Terminal_01x04, J6 Screw_Terminal_01x04, J7 Screw_Terminal_01x04, J8 Screw_Terminal_01x04, J9 Screw_Terminal_01x04, K1 SANYOU_SRD_Form_C, K10 SANYOU_SRD_Form_C, K11 SANYOU_SRD_Form_C, K12 SANYOU_SRD_Form_C, K13 SANYOU_SRD_Form_C, K14 SANYOU_SRD_Form_C, K15 SANYOU_SRD_Form_C, K16 SANYOU_SRD_Form_C, K17 SANYOU_SRD_Form_C, K18 SANYOU_SRD_Form_C, K19 SANYOU_SRD_Form_C, K2 SANYOU_SRD_Form_C, K20 SANYOU_SRD_Form_C, K21 SANYOU_SRD_Form_C, K22 SANYOU_SRD_Form_C, K23 SANYOU_SRD_Form_C, K24 SANYOU_SRD_Form_C, K3 SANYOU_SRD_Form_C, K4 SANYOU_SRD_Form_C, K5 SANYOU_SRD_Form_C, K6 SANYOU_SRD_Form_C, K7 SANYOU_SRD_Form_C, K8 SANYOU_SRD_Form_C, K9 SANYOU_SRD_Form_C, U1 MCP9808-E_SO8, U2 MCP9808-E_MS, U3 ULN2803A, U4 ULN2803A, U5 ULN2803A, U6 MCP23017_SS, U7 MCP23017_SS

Commit message: update
Parts:
- R6, R7: value 10k -> 4.7k
- renumbered A0 to JP1, A0 to JP10, A1 to JP2, A2 to JP3, A2 to JP5, A1 to JP6, A0 to JP7, A2 to JP8, A1 to JP9
Other:
- net class 230v removed
Changed lines of the file:
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@@
     (41 Cmts.User user)
     (42 Eco1.User user)
-    (43 Eco2.User user hide)
+    (43 Eco2.User user)
     (44 Edge.Cuts user)
     (45 Margin user)
@@
     (add_net K8)
     (add_net K9)
+    (add_net "Net-(J1-Pad1)")
+    (add_net "Net-(J1-Pad2)")
+    (add_net "Net-(J1-Pad3)")
+    (add_net "Net-(J1-Pad4)")
+    (add_net "Net-(J10-Pad1)")
+    (add_net "Net-(J10-Pad2)")
+    (add_net "Net-(J10-Pad3)")
+    (add_net "Net-(J10-Pad4)")
+    (add_net "Net-(J11-Pad1)")
+    (add_net "Net-(J11-Pad2)")
+    (add_net "Net-(J11-Pad3)")
+    (add_net "Net-(J11-Pad4)")
     (add_net "Net-(J12-Pad1)")
     (add_net "Net-(J12-Pad2)")
@@
     (add_net "Net-(J13-Pad3)")
     (add_net "Net-(J13-Pad4)")
+    (add_net "Net-(J2-Pad1)")
+    (add_net "Net-(J2-Pad2)")
+    (add_net "Net-(J2-Pad3)")
+    (add_net "Net-(J2-Pad4)")
+    (add_net "Net-(J4-Pad1)")
+    (add_net "Net-(J4-Pad2)")
+    (add_net "Net-(J4-Pad3)")
+    (add_net "Net-(J4-Pad4)")
+    (add_net "Net-(J5-Pad1)")
+    (add_net "Net-(J5-Pad2)")
+    (add_net "Net-(J5-Pad3)")
+    (add_net "Net-(J5-Pad4)")
     (add_net "Net-(J6-Pad1)")
     (add_net "Net-(J6-Pad2)")
@@
     (add_net "Net-(J7-Pad3)")
     (add_net "Net-(J7-Pad4)")
+    (add_net "Net-(J8-Pad1)")
+    (add_net "Net-(J8-Pad2)")
+    (add_net "Net-(J8-Pad3)")
+    (add_net "Net-(J8-Pad4)")
+    (add_net "Net-(J9-Pad1)")
+    (add_net "Net-(J9-Pad2)")
+    (add_net "Net-(J9-Pad3)")
+    (add_net "Net-(J9-Pad4)")
     (add_net "Net-(JP1-Pad2)")
     (add_net "Net-(JP10-Pad2)")
@@
     (uvia_drill 0.1)
   )
-  (net_class 230v ""
-    (clearance 1)
-    (trace_width 1)
-    (via_dia 1)
-    (via_drill 0.5)
-    (uvia_dia 0.3)
-    (uvia_drill 0.1)
-    (add_net "Net-(J1-Pad1)")
-    (add_net "Net-(J1-Pad2)")
-    (add_net "Net-(J1-Pad3)")
-    (add_net "Net-(J1-Pad4)")
-    (add_net "Net-(J10-Pad1)")
-    (add_net "Net-(J10-Pad2)")
-    (add_net "Net-(J10-Pad3)")
-    (add_net "Net-(J10-Pad4)")
-    (add_net "Net-(J11-Pad1)")
-    (add_net "Net-(J11-Pad2)")
-    (add_net "Net-(J11-Pad3)")
-    (add_net "Net-(J11-Pad4)")
-    (add_net "Net-(J2-Pad1)")
-    (add_net "Net-(J2-Pad2)")
-    (add_net "Net-(J2-Pad3)")
-    (add_net "Net-(J2-Pad4)")
-    (add_net "Net-(J4-Pad1)")
-    (add_net "Net-(J4-Pad2)")
-    (add_net "Net-(J4-Pad3)")
-    (add_net "Net-(J4-Pad4)")
-    (add_net "Net-(J5-Pad1)")
-    (add_net "Net-(J5-Pad2)")
-    (add_net "Net-(J5-Pad3)")
-    (add_net "Net-(J5-Pad4)")
-    (add_net "Net-(J8-Pad1)")
-    (add_net "Net-(J8-Pad2)")
-    (add_net "Net-(J8-Pad3)")
-    (add_net "Net-(J8-Pad4)")
-    (add_net "Net-(J9-Pad1)")
-    (add_net "Net-(J9-Pad2)")
-    (add_net "Net-(J9-Pad3)")
-    (add_net "Net-(J9-Pad4)")
-  )
   (module Relay_THT:Relay_SPDT_SANYOU_SRD_Series_Form_C (layer F.Cu)
     (at 460.5 296.908 90)
@@
   )
   (module Relay_THT:Relay_SPDT_SANYOU_SRD_Series_Form_C (layer F.Cu)
-    (at 443.71 296.908 90)
+    (at 443.73 296.908 90)
     (descr "relay Sanyou SRD series Form C http://www.sanyourelay.ca/public/products/pdf/SRD.pdf")
     (tags "relay Sanyu SRD form C")
@@
     (tags "solder jumper open")
     (attr virtual)
-    (fp_text reference A0 (at -2.78 0.1 270) (layer B.SilkS)
+    (fp_text reference JP10 (at -2.78 0.1 270) (layer B.SilkS)
       (effects (font (size 1 1) (thickness 0.15)) (justify mirror))
     )
@@
     (tags "solder jumper open")
     (attr virtual)
-    (fp_text reference A1 (at -2.78 0 270) (layer B.SilkS)
+    (fp_text reference JP9 (at -2.78 0 270) (layer B.SilkS)
       (effects (font (size 1 1) (thickness 0.15)) (justify mirror))
     )
@@
     (tags "solder jumper open")
     (attr virtual)
-    (fp_text reference A2 (at -2.78 -0.01 270) (layer B.SilkS)
+    (fp_text reference JP8 (at -2.78 -0.01 270) (layer B.SilkS)
       (effects (font (size 1 1) (thickness 0.15)) (justify mirror))
     )
@@
     (tags "solder jumper open")
     (attr virtual)
-    (fp_text reference A0 (at -2.97 0 270) (layer B.SilkS)
+    (fp_text reference JP7 (at -2.97 0 270) (layer B.SilkS)
       (effects (font (size 1 1) (thickness 0.15)) (justify mirror))
     )
@@
     (tags "solder jumper open")
     (attr virtual)
-    (fp_text reference A1 (at -2.97 0.04 270) (layer B.SilkS)
+    (fp_text reference JP6 (at -2.97 0.04 270) (layer B.SilkS)
       (effects (font (size 1 1) (thickness 0.15)) (justify mirror))
     )
@@
     (tags "solder jumper open")
     (attr virtual)
-    (fp_text reference A2 (at -2.97 0.07 270) (layer B.SilkS)
+    (fp_text reference JP5 (at -2.97 0.07 270) (layer B.SilkS)
       (effects (font (size 1 1) (thickness 0.15)) (justify mirror))
     )
@@
     (tags "solder jumper open")
     (attr virtual)
-    (fp_text reference A2 (at -2.8 0) (layer B.SilkS)
+    (fp_text reference JP3 (at -2.8 0) (layer B.SilkS)
       (effects (font (size 1 1) (thickness 0.15)) (justify mirror))
     )
@@
     (tags "solder jumper open")
     (attr virtual)
-    (fp_text reference A1 (at -2.8 0) (layer B.SilkS)
+    (fp_text reference JP2 (at -2.8 0) (layer B.SilkS)
       (effects (font (size 1 1) (thickness 0.15)) (justify mirror))
     )
@@
     (tags "solder jumper open")
     (attr virtual)
-    (fp_text reference A0 (at -2.8 0.01) (layer B.SilkS)
+    (fp_text reference JP1 (at -2.8 0.01) (layer B.SilkS)
       (effects (font (size 1 1) (thickness 0.15)) (justify mirror))
     )
@@
       (effects (font (size 1 1) (thickness 0.15)))
     )
-    (fp_text value 10k (at 0 1.43 90) (layer F.Fab)
+    (fp_text value 4.7k (at 0 1.43 90) (layer F.Fab)
       (effects (font (size 1 1) (thickness 0.15)))
     )
@@
       (effects (font (size 1 1) (thickness 0.15)))
     )
-    (fp_text value 10k (at 0 1.43 90) (layer F.Fab)
+    (fp_text value 4.7k (at 0 1.43 90) (layer F.Fab)
       (effects (font (size 1 1) (thickness 0.15)))
     )
