File: Circuit/boneIO - relay board 24x10A/boneIO - relay board.kicad_pcb (KiCad board)
At the start: 2 copper layers, 197 x 102 mm, 76 parts, among them J1 Screw_Terminal_01x04, J10 Screw_Terminal_01x04, J11 Screw_Terminal_01x04, J12 Screw_Terminal_01x04, J13 Screw_Terminal_01x04, J2 Screw_Terminal_01x04, J3 Conn_02x04_Odd_Even, J4 Screw_Terminal_01x04, J5 Screw_Terminal_01x04, J6 Screw_Terminal_01x04, J7 Screw_Terminal_01x04, J8 Screw_Terminal_01x04, J9 Screw_Terminal_01x04, K1 SANYOU_SRD_Form_C, K10 SANYOU_SRD_Form_C, K11 SANYOU_SRD_Form_C, K12 SANYOU_SRD_Form_C, K13 SANYOU_SRD_Form_C, K14 SANYOU_SRD_Form_C, K15 SANYOU_SRD_Form_C, K16 SANYOU_SRD_Form_C, K17 SANYOU_SRD_Form_C, K18 SANYOU_SRD_Form_C, K19 SANYOU_SRD_Form_C, K2 SANYOU_SRD_Form_C, K20 SANYOU_SRD_Form_C, K21 SANYOU_SRD_Form_C, K22 SANYOU_SRD_Form_C, K23 SANYOU_SRD_Form_C, K24 SANYOU_SRD_Form_C, K3 SANYOU_SRD_Form_C, K4 SANYOU_SRD_Form_C, K5 SANYOU_SRD_Form_C, K6 SANYOU_SRD_Form_C, K7 SANYOU_SRD_Form_C, K8 SANYOU_SRD_Form_C, K9 SANYOU_SRD_Form_C, U1 MCP9808-E_SO8, U2 MCP9808-E_MS, U3 ULN2803A, U4 ULN2803A, U5 ULN2803A, U6 MCP23017_SS, U7 MCP23017_SS

Commit message: Update
Parts:
- renumbered JP10 to A0, JP7 to A0, JP1 to A0, JP9 to A1, JP6 to A1, JP2 to A1, JP8 to A2, JP5 to A2, JP3 to A2
Other:
- board text added: "DOWN"
- board text added: "WARNING!!!"
