File: Circuit/boneIO - relay board 24x10A/boneIO - relay board.sch (KiCad schematic (older format))
At the start: 75 parts, among them J1 Screw_Terminal_01x04, J10 Screw_Terminal_01x04, J11 Screw_Terminal_01x04, J12 Screw_Terminal_01x04, J13 Screw_Terminal_01x04, J2 Screw_Terminal_01x04, J3 Conn_02x04_Odd_Even, J4 Screw_Terminal_01x04, J5 Screw_Terminal_01x04, J6 Screw_Terminal_01x04, J7 Screw_Terminal_01x04, J8 Screw_Terminal_01x04, J9 Screw_Terminal_01x04, K1 SANYOU_SRD_Form_C, K10 SANYOU_SRD_Form_C, K11 SANYOU_SRD_Form_C, K12 SANYOU_SRD_Form_C, K13 SANYOU_SRD_Form_C, K14 SANYOU_SRD_Form_C, K15 SANYOU_SRD_Form_C, K16 SANYOU_SRD_Form_C, K17 SANYOU_SRD_Form_C, K18 SANYOU_SRD_Form_C, K19 SANYOU_SRD_Form_C, K2 SANYOU_SRD_Form_C, K20 SANYOU_SRD_Form_C, K21 SANYOU_SRD_Form_C, K22 SANYOU_SRD_Form_C, K23 SANYOU_SRD_Form_C, K24 SANYOU_SRD_Form_C, K3 SANYOU_SRD_Form_C, K4 SANYOU_SRD_Form_C, K5 SANYOU_SRD_Form_C, K6 SANYOU_SRD_Form_C, K7 SANYOU_SRD_Form_C, K8 SANYOU_SRD_Form_C, K9 SANYOU_SRD_Form_C, U1 MCP9808-E_SO8, U2 MCP9808-E_MS, U3 ULN2803A, U4 ULN2803A, U5 ULN2803A, U6 MCP23017_SS, U7 MCP23017_SS

Commit message: update
Parts:
- R6, R7: value 10k -> 4.7k
Other:
- note added: "- relay board 24x10A v0.1"
- note removed: "- relay board 24x12A v0.1"
Changed lines of the file:
@@
 P 7000 4750
 F 0 "R7" H 7070 4796 50  0000 L CNN
-F 1 "10k" H 7070 4705 50  0000 L CNN
+F 1 "4.7k" H 7070 4705 50  0000 L CNN
 F 2 "Resistor_SMD:R_0603_1608Metric" V 6930 4750 50  0001 C CNN
 F 3 "~" H 7000 4750 50  0001 C CNN
@@
 P 7000 4450
 F 0 "R6" H 7070 4496 50  0000 L CNN
-F 1 "10k" H 7070 4405 50  0000 L CNN
+F 1 "4.7k" H 7070 4405 50  0000 L CNN
 F 2 "Resistor_SMD:R_0603_1608Metric" V 6930 4450 50  0001 C CNN
 F 3 "~" H 7000 4450 50  0001 C CNN
@@
 MCP23017
 Text Notes 10200 1150 0    197  ~ 39
-- relay board 24x12A v0.1
+- relay board 24x10A v0.1
 NoConn ~ 18700 3650
 NoConn ~ 18700 3750
